File: hardware/LabnodeIO/LabnodeIO.kicad_pcb (KiCad board)
At the start: 2 copper layers, 17 parts, among them J1 mc 0.5-2.5, J2 EXT3, J3 mc 0.5-2.5, U1 PCF8574, U2 LM324

Commit message: layout labnodeIO
Parts:
- C3, D1, D2, J1, J2, J3: moved to B.Cu
- moved D1 59.0 mm to (52.0, 46.0), turned to 270 degrees
- moved R4 55.4 mm to (55.5, 55.1), turned to 270 degrees
- moved D2 55.2 mm to (52.0, 56.0), turned to 90 degrees
- moved U2 53.8 mm to (65.0, 51.0)
- moved J1 53.4 mm to (73.0, 18.0), turned to 270 degrees
- moved R1 52.9 mm to (59.0, 47.0), turned to 270 degrees
- moved J2 52.7 mm to (39.0, 40.5), turned to 180 degrees
- moved R7 52.2 mm to (49.0, 55.0), turned to 270 degrees
- moved R5 51.2 mm to (53.6, 42.5), turned to 180 degrees
- moved C3 50.9 mm to (65.0, 43.0), turned to 180 degrees
- moved J3 49.1 mm to (72.0, 50.0), turned to 270 degrees
- moved R2 49.0 mm to (55.5, 47.1), turned to 90 degrees
- moved R3 48.4 mm to (59.0, 55.1), turned to 90 degrees
- moved C2 45.3 mm to (45.5, 55.0), turned to 270 degrees
- moved R6 42.2 mm to (49.0, 47.0), turned to 90 degrees
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Connections:
- J1 pad 1: Net-(J1-Pad1) -> +12V
- J1 pad 10: (no net) -> Net-(J1-Pad10)
- J1 pad 2: Net-(J1-Pad2) -> +12V
- J1 pad 9: +12V -> Net-(J1-Pad9)
- U1 pad 10: Net-(J1-Pad6) -> Net-(J1-Pad5)
- U1 pad 11: Net-(J1-Pad7) -> Net-(J1-Pad4)
- U1 pad 12: Net-(J1-Pad8) -> Net-(J1-Pad3)
- U1 pad 4: Net-(J1-Pad1) -> Net-(J1-Pad10)
- U1 pad 5: Net-(J1-Pad2) -> Net-(J1-Pad9)
- U1 pad 6: Net-(J1-Pad3) -> Net-(J1-Pad8)
- U1 pad 7: Net-(J1-Pad4) -> Net-(J1-Pad7)
- U1 pad 9: Net-(J1-Pad5) -> Net-(J1-Pad6)
Routing:
- net GND: track 0.00 -> 61.8 mm
- net Net-(J1-Pad3): track 0.00 -> 40.8 mm
- net Net-(J1-Pad4): track 0.00 -> 36.2 mm
- net Net-(J3-Pad3): track 0.00 -> 33.8 mm
- net Net-(J1-Pad5): track 0.00 -> 32.1 mm
- net +12V: track 0.00 -> 28.2 mm
- net Net-(J1-Pad6): track 0.00 -> 25.2 mm
- net analog1: track 0.00 -> 20.5 mm
- net analog0: track 0.00 -> 20.5 mm
- net Net-(J3-Pad2): track 0.00 -> 18.2 mm
- net Net-(J1-Pad10): track 0.00 -> 14.3 mm
- net Net-(J1-Pad9): track 0.00 -> 13.8 mm
- net Net-(J1-Pad8): track 0.00 -> 13.3 mm
- net Net-(J1-Pad7): track 0.00 -> 12.7 mm
- net Net-(R5-Pad1): track 0.00 -> 10.6 mm
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- added copper zone on F.Cu, net GND

Commit message: layout fertig
Parts:
- moved C1 25.5 mm to (44.0, 21.5)
- moved D1 25.5 mm to (50.5, 20.5)
- moved D2 25.5 mm to (50.5, 30.5)
- moved J3 25.5 mm to (70.5, 24.5)
- moved R1 25.5 mm to (57.5, 21.5)
- moved R2 25.5 mm to (54.0, 21.6)
- moved R3 25.5 mm to (57.5, 29.6)
- moved R4 25.5 mm to (54.0, 29.6)
- moved R6 25.5 mm to (47.5, 21.5)
- moved R7 25.5 mm to (47.5, 29.5)
- moved U2 25.5 mm to (63.5, 25.5)
- moved C2 22.8 mm to (53.0, 33.5), turned to 0 degrees
- moved C3 16.7 mm to (54.0, 55.5), turned to 90 degrees
- moved J1 16.2 mm to (70.5, 34.0)
- moved R5 12.5 mm to (58.6, 54.0)
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Connections:
- J1 pad 1: +12V -> Net-(J1-Pad1)
- J1 pad 10: Net-(J1-Pad10) -> +12V
- J1 pad 2: +12V -> Net-(J1-Pad2)
- J1 pad 9: Net-(J1-Pad9) -> +12V
- J2 pad 10: (no net) -> +12V
- U1 pad 10: Net-(J1-Pad5) -> Net-(J1-Pad3)
- U1 pad 11: Net-(J1-Pad4) -> Net-(J1-Pad2)
- U1 pad 12: Net-(J1-Pad3) -> Net-(J1-Pad1)
- U1 pad 4: Net-(J1-Pad10) -> Net-(J1-Pad8)
- U1 pad 5: Net-(J1-Pad9) -> Net-(J1-Pad7)
- U1 pad 6: Net-(J1-Pad8) -> Net-(J1-Pad6)
- U1 pad 7: Net-(J1-Pad7) -> Net-(J1-Pad5)
- U1 pad 9: Net-(J1-Pad6) -> Net-(J1-Pad4)
Routing:
- net +12V: track 28.2 -> 74.9 mm, vias 0 -> 4
- net Net-(J1-Pad1): track 0.00 -> 29.6 mm
- net Net-(J1-Pad5): track 32.1 -> 5.53 mm
- net Net-(J1-Pad2): track 0.00 -> 25.5 mm
- net analog1: track 20.5 -> 42.6 mm
- net analog0: track 20.5 -> 41.2 mm
- net Net-(J1-Pad4): track 36.2 -> 16.4 mm
- net Net-(J1-Pad6): track 25.2 -> 6.05 mm
- net Net-(J1-Pad3): track 40.8 -> 21.8 mm
- net Net-(J1-Pad10): track 14.3 -> 0.00 mm
- net Net-(J1-Pad9): track 13.8 -> 0.00 mm
- net SCL: track 0.00 -> 13.6 mm
- net SDA: track 0.00 -> 11.2 mm
- net +5V: track 4.23 -> 14.9 mm
- net Net-(J1-Pad7): track 12.7 -> 6.55 mm
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Other:
- net class Default: clearance 0.2 -> 0.4; trace_width 0.25 -> 0.5; via_dia 0.6 -> 1.5; via_drill 0.4 -> 1
- rule trace_clearance: 0.2 -> 0.4

Commit message: Ausgangskondensatoren eingefügt
Parts:
- added C4: 100u, Capacitors_THT:CP_Radial_D4.0mm_P2.00mm, B.Cu at (72.5, 19.0)
- added C5: 100u, Capacitors_THT:CP_Radial_D4.0mm_P2.00mm, B.Cu at (60.5, 31.5)
- moved C1 8.50 mm to (52.5, 21.5)
- moved D1 3.61 mm to (47.5, 22.5), turned to 90 degrees
- moved R7 3.00 mm to (50.5, 29.6)
- moved D2 3.00 mm to (47.5, 30.5)
- moved R6 2.50 mm to (50.0, 21.6)
- moved R2 1.00 mm to (55.0, 21.5)
Routing:
- net analog0: track 41.2 -> 44.0 mm
- net Net-(C4-Pad1): track 28.9 -> 30.7 mm
- net Net-(D1-Pad1): track 3.87 -> 2.58 mm
- net GND: track 61.7 -> 60.7 mm
- net Net-(R1-Pad2): track 6.99 -> 6.09 mm
- net analog1: track 42.6 -> 41.9 mm

Commit message: 5v auf stecker
Connections:
- J1 pad 9: +12V -> +5V
Routing:
- net GND: track 60.7 -> 110.5 mm, vias 2 -> 6
- net +5V: track 14.9 -> 30.1 mm
Changed lines of the file:
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@@
   (general
     (links 50)
-    (no_connects 3)
-    (area 39.899999 15.224999 77.085 60.600001)
+    (no_connects 0)
+    (area 0 0 0 0)
     (thickness 1.6)
     (drawings 4)
-    (tracks 166)
+    (tracks 191)
     (zones 0)
     (modules 19)
@@
     (mod_text_size 1 1)
     (mod_text_width 0.15)
-    (pad_size 2 2)
+    (pad_size 2 1)
     (pad_drill 1)
     (pad_to_mask_clearance 0.2)
@@
     (visible_elements FFFFEF7F)
     (pcbplotparams
-      (layerselection 0x00030_80000001)
+      (layerselection 0x00000_00000001)
       (usegerberextensions false)
       (excludeedgelayer true)
@@
       (padsonsilk false)
       (subtractmaskfromsilk false)
-      (outputformat 1)
+      (outputformat 4)
       (mirror false)
-      (drillshape 1)
+      (drillshape 0)
       (scaleselection 1)
       (outputdirectory ""))
@@
       (net 12 "Net-(J1-Pad8)"))
     (pad 9 thru_hole oval (at 20 0 270) (size 2 2) (drill 1) (layers *.Cu *.Mask)
-      (net 4 +12V))
+      (net 13 +5V))
     (pad 10 thru_hole oval (at 22.54 0 270) (size 2 2) (drill 1) (layers *.Cu *.Mask)
       (net 4 +12V))
@@
       (effects (font (size 1 1) (thickness 0.15)) (justify mirror))
     )
-    (pad 1 thru_hole rect (at 0 0) (size 1 1) (drill 1) (layers *.Cu *.Mask)
-      (net 2 GND))
-    (pad 2 thru_hole oval (at 2 0) (size 1 1) (drill 1) (layers *.Cu *.Mask)
+    (pad 1 thru_hole rect (at 0 0) (size 2 1) (drill 1 (offset -0.5 0)) (layers *.Cu *.Mask)
+      (net 2 GND))
+    (pad 2 thru_hole oval (at 2 0) (size 2 1) (drill 1 (offset 0.5 0)) (layers *.Cu *.Mask)
       (net 13 +5V))
-    (pad 3 thru_hole oval (at 0 -2.54) (size 1 1) (drill 1) (layers *.Cu *.Mask)
+    (pad 3 thru_hole oval (at 0 -2.54) (size 2 1) (drill 1 (offset -0.5 0)) (layers *.Cu *.Mask)
       (net 14 SCL))
-    (pad 4 thru_hole oval (at 2 -2.54) (size 1 1) (drill 1) (layers *.Cu *.Mask)
+    (pad 4 thru_hole oval (at 2 -2.54) (size 2 1) (drill 1 (offset 0.5 0)) (layers *.Cu *.Mask)
       (net 15 SDA))
-    (pad 5 thru_hole oval (at 0 -5) (size 1 1) (drill 1) (layers *.Cu *.Mask)
+    (pad 5 thru_hole oval (at 0 -5) (size 2 1) (drill 1 (offset -0.5 0)) (layers *.Cu *.Mask)
       (net 1 analog0))
-    (pad 6 thru_hole oval (at 2 -5) (size 1 1) (drill 1) (layers *.Cu *.Mask)
+    (pad 6 thru_hole oval (at 2 -5) (size 2 1) (drill 1 (offset 0.5 0)) (layers *.Cu *.Mask)
       (net 3 analog1))
     (pad 7 thru_hole oval (at 0 -7.54) (size 1 1) (drill 1) (layers *.Cu *.Mask))
     (pad 8 thru_hole oval (at 2 -7.54) (size 1 1) (drill 1) (layers *.Cu *.Mask))
     (pad 9 thru_hole oval (at 0 -10) (size 1 1) (drill 1) (layers *.Cu *.Mask))
-    (pad 10 thru_hole oval (at 2 -10) (size 1 1) (drill 1) (layers *.Cu *.Mask)
+    (pad 10 thru_hole oval (at 2 -10) (size 2 1) (drill 1 (offset 0.5 0)) (layers *.Cu *.Mask)
       (net 4 +12V))
     (model ${KISYS3DMOD}/Pin_Headers.3dshapes/Pin_Header_Straight_2x05_Pitch2.54mm.wrl
@@
   )
   (gr_line (start 40 60.5) (end 40 15.5) (layer Margin) (width 0.2))
-  (gr_line (start 75 60.5) (end 40 60.5) (layer Margin) (width 0.2))
-  (gr_line (start 75 15.5) (end 75 60.5) (layer Margin) (width 0.2))
-  (gr_line (start 40 15.5) (end 75 15.5) (layer Margin) (width 0.2))
+  (gr_line (start 79 60.5) (end 40 60.5) (layer Margin) (width 0.2))
+  (gr_line (start 79 15.5) (end 79 60.5) (layer Margin) (width 0.2))
+  (gr_line (start 40 15.5) (end 79 15.5) (layer Margin) (width 0.2))
   (segment (start 44.73 24.23) (end 45.5 24.23) (width 0.5) (layer F.Cu) (net 1))
   (segment (start 45.5 24.23) (end 52.23 24.23) (width 0.5) (layer F.Cu) (net 1))
@@
   (segment (start 43 41.5) (end 44.5 43) (width 0.5) (layer F.Cu) (net 1))
   (segment (start 60.8 24.23) (end 52.23 24.23) (width 0.5) (layer F.Cu) (net 1))
+  (segment (start 64.77 59.69) (end 62.23 59.69) (width 0.5) (layer F.Cu) (net 2))
+  (segment (start 62.23 59.69) (end 45.72 59.69) (width 0.5) (layer F.Cu) (net 2))
+  (segment (start 62.23 53.34) (end 62.23 59.69) (width 0.5) (layer B.Cu) (net 2))
+  (via (at 62.23 59.69) (size 1.5) (drill 1) (layers F.Cu B.Cu) (net 2))
+  (segment (start 64.77 53.34) (end 62.23 53.34) (width 0.5) (layer F.Cu) (net 2))
+  (via (at 62.23 53.34) (size 1.5) (drill 1) (layers F.Cu B.Cu) (net 2))
+  (segment (start 45.72 59.69) (end 44.5 58.47) (width 0.5) (layer F.Cu) (net 2))
+  (segment (start 44.5 58.47) (end 44.5 48) (width 0.5) (layer F.Cu) (net 2))
+  (segment (start 64.77 53.34) (end 64.77 59.69) (width 0.5) (layer B.Cu) (net 2))
+  (via (at 64.77 59.69) (size 1.5) (drill 1) (layers F.Cu B.Cu) (net 2))
+  (segment (start 65.5 50.31) (end 65.5 52.61) (width 0.5) (layer F.Cu) (net 2))
+  (segment (start 65.5 52.61) (end 64.77 53.34) (width 0.5) (layer F.Cu) (net 2))
+  (via (at 64.77 53.34) (size 1.5) (drill 1) (layers F.Cu B.Cu) (net 2))
   (segment (start 72.5 17) (end 71.5 17) (width 0.5) (layer F.Cu) (net 2))
   (segment (start 71.5 17) (end 69.5 19) (width 0.5) (layer F.Cu) (net 2))
@@
   (segment (start 48.5 43) (end 46.5 43) (width 0.5) (layer F.Cu) (net 3))
   (segment (start 60.8 26.77) (end 52.23 26.77) (width 0.5) (layer F.Cu) (net 3))
-  (segment (start 48 36) (end 46.5 36) (width 0.5) (layer F.Cu) (net 4))
+  (segment (start 46.5 38) (end 46.5 37.5) (width 0.5) (layer F.Cu) (net 4))
+  (segment (start 46.5 37.5) (end 48 36) (width 0.5) (layer F.Cu) (net 4))
+  (segment (start 46.5 36) (end 46.5 38) (width 0.5) (layer F.Cu) (net 4))
+  (segment (start 54.65 57.15) (end 68.435787 57.15) (width 0.5) (layer F.Cu) (net 4))
+  (segment (start 68.435787 57.15) (end 69.085787 56.5) (width 0.5) (layer F.Cu) (net 4))
+  (segment (start 69.085787 56.5) (end 70.5 56.5) (width 0.5) (layer F.Cu) (net 4))
+  (segment (start 54 55.5) (end 54 56.5) (width 0.5) (layer F.Cu) (net 4))
+  (segment (start 54 56.5) (end 54.65 57.15) (width 0.5) (layer F.Cu) (net 4))
   (segment (start 51.5 36) (end 48 36) (width 0.5) (layer B.Cu) (net 4))
   (via (at 48 36) (size 1.5) (drill 1) (layers F.Cu B.Cu) (net 4))
@@
   (segment (start 53 55.5) (end 51.5 54) (width 0.5) (layer F.Cu) (net 4))
   (via (at 51.5 54) (size 1.5) (drill 1) (layers F.Cu B.Cu) (net 4))
-  (segment (start 70.5 56.5) (end 55 56.5) (width 0.5) (layer F.Cu) (net 4))
-  (segment (start 55 56.5) (end 54 55.5) (width 0.5) (layer F.Cu) (net 4))
   (segment (start 44.59999 32.372796) (end 46.5 34.272806) (width 0.5) (layer F.Cu) (net 4))
   (segment (start 46.5 34.272806) (end 46.5 36) (width 0.5) (layer F.Cu) (net 4))
@@
   (segment (start 44.59999 26.90001) (end 44.59999 32.372796) (width 0.5) (layer F.Cu) (net 4))
   (segment (start 60.8 25.5) (end 46 25.5) (width 0.5) (layer F.Cu) (net 4))
-  (segment (start 46.5 38) (end 46.5 36) (width 0.5) (layer F.Cu) (net 4))
-  (segment (start 70.5 56.5) (end 70.5 53.96) (width 0.5) (layer F.Cu) (net 4))
   (segment (start 47.5 22.5) (end 49.8 22.5) (width 0.5) (layer F.Cu) (net 5))
   (segment (start 49.8 22.5) (end 50 22.7) (width 0.5) (layer F.Cu) (net 5))
@@
   (segment (start 68.749999 49.749999) (end 69.500001 50.500001) (width 0.5) (layer F.Cu) (net 12))
   (segment (start 69.500001 50.500001) (end 70.5 51.5) (width 0.5) (layer F.Cu) (net 12))
+  (segment (start 57.5 54) (end 57.5 54.96) (width 0.5) (layer F.Cu) (net 13))
+  (segment (start 57.5 54.96) (end 58.42 55.88) (width 0.5) (layer F.Cu) (net 13))
+  (segment (start 58.42 55.88) (end 67.31 55.88) (width 0.5) (layer F.Cu) (net 13))
+  (segment (start 67.31 55.88) (end 68.58 54.61) (width 0.5) (layer F.Cu) (net 13))
+  (segment (start 68.58 54.61) (end 68.58 54.465787) (width 0.5) (layer F.Cu) (net 13))
+  (segment (start 68.58 54.465787) (end 69.085787 53.96) (width 0.5) (layer F.Cu) (net 13))
+  (segment (start 69.085787 53.96) (end 70.5 53.96) (width 0.5) (layer F.Cu) (net 13))
   (segment (start 46.5 48) (end 48.81 50.31) (width 0.5) (layer F.Cu) (net 13))
   (segment (start 48.81 50.31) (end 56.2 50.31) (width 0.5) (layer F.Cu) (net 13))
   (segment (start 56.2 50.31) (end 56.2 52.7) (width 0.5) (layer F.Cu) (net 13))
   (segment (start 56.2 52.7) (end 57.5 54) (width 0.5) (layer F.Cu) (net 13))
-  (segment (start 47.809999 44.309999) (end 51.27 47.77) (width 0.5) (layer F.Cu) (net 14))
-  (segment (start 51.27 47.77) (end 56.2 47.77) (width 0.5) (layer F.Cu) (net 14))
   (segment (start 44.5 45.46) (end 45.650001 44.309999) (width 0.5) (layer F.Cu) (net 14))
-  (segment (start 45.650001 44.309999) (end 47.809999 44.309999) (width 0.5) (layer F.Cu) (net 14))
-  (segment (start 46.5 45.46) (end 50.08 49.04) (width 0.5) (layer F.Cu) (net 15))
-  (segment (start 50.08 49.04) (end 56.2 49.04) (width 0.5) (layer F.Cu) (net 15))
+  (segment (start 45.650001 44.309999) (end 48.237997 44.309999) (width 0.5) (layer F.Cu) (net 14))
+  (segment (start 48.237997 44.309999) (end 51.697998 47.77) (width 0.5) (layer F.Cu) (net 14))
+  (segment (start 51.697998 47.77) (end 54.95 47.77) (width 0.5) (layer F.Cu) (net 14))
+  (segment (start 54.95 47.77) (end 56.2 47.77) (width 0.5) (layer F.Cu) (net 14))
+  (segment (start 48 45.46) (end 51.58 49.04) (width 0.5) (layer F.Cu) (net 15))
+  (segment (start 51.58 49.04) (end 56.2 49.04) (width 0.5) (layer F.Cu) (net 15))
+  (segment (start 46.5 45.46) (end 48 45.46) (width 0.5) (layer F.Cu) (net 15))
   (segment (start 55 22.6) (end 57.5 22.6) (width 0.5) (layer F.Cu) (net 16))
   (segment (start 57.4 22.7) (end 57.5 22.6) (width 0.5) (layer F.Cu) (net 16))
@@
     (polygon
       (pts
-        (xy 40 15.5) (xy 75 15.5) (xy 75 60.5) (xy 40 60.5)
+        (xy 40 15.5) (xy 79 15.5) (xy 79 60.5) (xy 40 60.5)
       )
     )
