File: hardware/LabnodeIO-XL/file5A949986.sch (KiCad schematic (older format))
At the start: 25 parts, among them U3 LM324

Commit message: Platinenlayout und 3d modell angefangen
Parts:
- removed C1, C2, C4, C5: 100u, Capacitors_THT:CP_Radial_D4.0mm_P2.00mm, symbol C_Small
- removed D1, D2, D3, D4: LED_Small, LEDs:LED_D3.0mm, symbol LED_Small
- removed R1, R2, R3, R4: R, Resistors_SMD:R_0603_HandSoldering, symbol R_Small
- C6, C7, C8, C9: footprint Capacitors_SMD:C_0805_HandSoldering -> Capacitors_SMD:C_0603
- R10, R11, R12, R13, R6, R7, R8, R9: footprint Resistors_SMD:R_0603_HandSoldering -> Resistors_SMD:R_0603
- U3: footprint (none) -> Housings_SOIC:SOIC-14_3.9x8.7mm_Pitch1.27mm
Connections:
- wire segments 72 -> 66

Commit message: eingangswiderstände hinzugefuegt und geroutet
Parts:
- added R26, R27, R28, R4: 22k, Resistors_SMD:R_0603, symbol R_Small
Connections:
- wire segments 66 -> 52
