File: hardware/LabnodeCAN/LabnodeCAN.sch (KiCad schematic (older format))
At the start: 47 parts, among them J1 USB_B_Mini, J2 CAN, J3 PWR, J4 ISP, J5 EXTa, J6 EXTb, U1 ATMEGA32-16AU, U2 MCP2515-EST, U3 LM2574M-5, U4 MCP2551-I-SN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

Commit message: LabnodeCAN cvpcb finished
Parts:
- removed J1: USB_B_Mini, symbol Connector_Specialized:USB_B_Mini
- added J1: USB_B_Micro, LabnodeCAN:USB_Micro-B_Amphenol_10118194-0001LF_Horizontal, symbol Connector_Specialized:USB_B_Micro
- C1, C11, C13, C2, C3, C4, C5, C6, C8, C9: footprint (none) -> Capacitor_SMD:C_0603_1608Metric
- C10: footprint (none) -> Capacitor_SMD:CP_Elec_8x10.5
- C12: footprint (none) -> Capacitor_SMD:CP_Elec_4x5.7
- C7: footprint (none) -> Capacitor_SMD:CP_Elec_6.3x5.7
- D1, D2: footprint (none) -> Diode_SMD:D_SOT-23_ANK
- D3, D6: footprint (none) -> LED_SMD:LED_0603_1608Metric
- D4: footprint (none) -> Diode_SMD:D_MELF
- D5: footprint (none) -> Diode_THT:D_DO-41_SOD81_P7.62mm_Horizontal
- J2, J4: footprint (none) -> Connector_PinHeader_2.54mm:PinHeader_2x05_P2.54mm_Vertical
- J3: footprint (none) -> Connector_BarrelJack:BarrelJack_CUI_PJ-102AH_Horizontal
- J5, J6: footprint (none) -> Connector_PinHeader_2.54mm:PinHeader_1x15_P2.54mm_Vertical
- JP1, JP2: footprint (none) -> Connector_PinHeader_2.54mm:PinHeader_1x03_P2.54mm_Vertical
- L1: value L -> 10µ
- R1, R10, R11, R12, R2, R3, R4, R5, R6, R7, R8, R9: footprint (none) -> Resistor_SMD:R_0603_1608Metric

Commit message: e7p's status...
Parts:
- removed J5: EXTa, Connector_PinHeader_2.54mm:PinHeader_1x15_P2.54mm_Vertical, symbol Connector_Generic:Conn_01x15
- removed J6: EXTb, Connector_PinHeader_2.54mm:PinHeader_1x15_P2.54mm_Vertical, symbol Connector_Generic:Conn_01x15
- added C14: 1u, Capacitor_SMD:C_0603_1608Metric, symbol Device:C
- added C15, C16: 1u, Capacitor_SMD:C_0603_1608Metric, symbol Device:CP
- added C17: 2u, Capacitor_SMD:C_0603_1608Metric, symbol Device:C
- added C18: 10u, Capacitor_SMD:C_0603_1608Metric, symbol Device:C
- added C19: 100n, Capacitor_SMD:C_0603_1608Metric, symbol Device:C
- added D7: 1N4148, Diode_SMD:D_MELF, symbol Device:D
- added J5: Conn_02x17_Odd_Even, Connector_PinHeader_2.54mm:PinHeader_2x17_P2.54mm_Vertical, symbol Connector_Generic:Conn_02x17_Odd_Even
- added J6: Conn_02x02_Odd_Even, Connector_PinHeader_2.54mm:PinHeader_2x02_P2.54mm_Vertical, symbol Connector_Generic:Conn_02x02_Odd_Even
- added R13: 390k, Resistor_SMD:R_0603_1608Metric, symbol Device:R
- added R14: 4k7, Resistor_SMD:R_0603_1608Metric, symbol Device:R
- added U6: SSD1306, LabnodeCAN:SSD1306_128x64_backmount, symbol SSD1306:SSD1306
- J2, J4: footprint Connector_PinHeader_2.54mm:PinHeader_2x05_P2.54mm_Vertical -> Connector_IDC:IDC-Header_2x05_P2.54mm_Vertical
- L1: footprint (none) -> Inductor_SMD:L_0603_1608Metric
- L2: footprint (none) -> LabnodeCAN:L_SMD_95_90
- R5: footprint Resistor_SMD:R_0603_1608Metric -> Resistor_SMD:R_1206_3216Metric
- Y1: footprint (none) -> Crystal:Crystal_SMD_HC49-SD
Connections:
- net labels added: PC4, PC5, PC6, PC7
- wire segments 288 -> 392
- no-connect marks 12 -> 8
Other:
- moved on the sheet: J3, U3
